File: hardware/ICARUS_1U_Solar_Panel_PCB_v0p4.kicad_sch (KiCad schematic)
At the start: 4 parts, among them J1 Molex_53398-0471

Commit message: Fix v0.4 schematic annotation by using numeric TVS reference
Parts:
- renumbered D_TVS_DNP to D1
Changed lines of the file:
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@@
 	)
 	(symbol (lib_id "ICARUS:TVS_DNP_2Pin") (at 130.81 106.5 0) (unit 1) (exclude_from_sim no) (in_bom no) (on_board yes) (dnp yes)
-		(property "Reference" "D_TVS_DNP" (at 130.81 101.0 0) (effects (font (size 1.27 1.27))))
+		(property "Reference" "D1" (at 130.81 101.0 0) (effects (font (size 1.27 1.27))))
 		(property "Value" "TVS_OPTIONAL_DNP" (at 130.81 112.0 0) (effects (font (size 1.27 1.27))))
 		(property "Footprint" "Diode_SMD:D_SOD-123" (at 130.81 115.0 0) (effects (font (size 1.27 1.27)) hide))
