File: hardware/ICARUS_1U_Solar_Panel_PCB_v0p6.kicad_pcb (KiCad board)
At the start: 2 copper layers, 95 x 95 mm, 13 parts, among them J1 Molex_53398-0471

Commit message: Fix anti-series cell topology and reroute board to clean DRC
The two cells were physically in anti-series (both back/+ contacts tied to SERIES_MID), which schematic-parity cannot detect. Corrected SC2 pad numbering and net assignment so the panel is a true 2S series (SERIES_MID = SC1 back + SC2 tabs), moved both back-contact pads to F.Cu, moved D1 (DNP) clear of the routing, and rebuilt all routing. KiCad 10 DRC with schematic parity: 0 errors, 0 unconnected, 0 shorts, 0 parity problems; remaining 13 are library-resolution warnings (waived). Adds CORRECAO_TOPOLOGIA_SERIE_v0p6.md and regenerates reports/plots.

Cell back-contact scheme, tab geometry and D1 placement remain provisional pending the vendor CIC assembly drawing.

Co-Authored-By: Claude Opus 4.7 (1M context) <noreply@anthropic.com>
Parts:
- moved D1 13.6 mm to (120.0, 138.0)
Routing:
- net PANEL_POS: track 105.1 -> 171.7 mm, vias 0 -> 3
- net PANEL_NEG: track 247.6 -> 274.6 mm
- net SERIES_MID: track 189.7 -> 200.1 mm, vias 1 -> 3
