File: hardware/ICARUS_1U_Solar_Panel_PCB_v0p7.kicad_pcb (KiCad board)
At the start: 2 copper layers, 95 x 95 mm, 13 parts, among them J1 Molex_53398-0471

Commit message: Switch to parallel topology (1S2P) for v0.7
Lead-team-driven topology change. Both cells now share PANEL_POS and
PANEL_NEG nets (was 2S1P with intermediate SERIES_MID). J1 (Molex)
moved from F.Cu to B.Cu (bottom side, as instructed). Re-routed for
parallel: left B.Cu corridor (x=70) ties the two PANEL_NEG tab buses;
right B.Cu corridor (x=137) ties the two PANEL_POS centre buses; both
land on the bottom J1 pads. TP3/TP5 stay on F.Cu under SC2 (PANEL_POS
on PANEL_POS) to avoid crossing the B.Cu PANEL_NEG corridor.

Also removed: D1 (TVS DNP) and TP2 (SERIES_MID test pad), both obsolete
in 1S2P. SERIES_MID net dropped from the PCB net table.

Rename of v0p6.* -> v0p7.* across .kicad_sch / .kicad_pcb / .kicad_pro.

DRC parity clean: 0 errors / 0 unconnected / 0 parity / 0 shorts.
11 warnings = same library waivers as v0.6 (minus the D1/TP2 ones).

Co-Authored-By: Claude Opus 4.7 <noreply@anthropic.com>
Parts:
- removed D1: TVS_OPTIONAL_DNP, Diode_SMD:D_SOD-123
- removed TP2: SERIES_MID, TestPoint:TestPoint_Pad_D2.0mm
- J1: moved to B.Cu
Connections:
- SC1 pad 2: SERIES_MID -> PANEL_POS
- SC2 pad 1: SERIES_MID -> PANEL_NEG
Routing:
- net SERIES_MID: track 200.1 -> 0.00 mm, vias 3 -> 0
- net PANEL_POS: track 171.7 -> 261.8 mm, vias 3 -> 2
- net PANEL_NEG: track 274.6 -> 326.1 mm, vias 4 -> 2

Commit message: Fix outdated board silkscreen labels for v0.7
Two leftover cosmetic strings from the 2S1P baseline that were still
showing in the KiCad GUI:
- Board title: "2S1P BASELINE" -> "1S2P PARALLEL"
- Test-point legend: "TP: PV- / MID / PV+" -> "TP: PV- / PV+" (TP2 was
  removed with the SERIES_MID net)

DRC parity still clean (0 errors / 0 unconnected / 0 parity).

Co-Authored-By: Claude Opus 4.7 <noreply@anthropic.com>
Other:
- board text added: "ICARUS - 1U SOLAR PANEL PCB - 1S2P PARALLEL"
- board text added: "TP: PV- / PV+"
- board text removed: "ICARUS - 1U SOLAR PANEL PCB - 2S1P BASELINE"
- board text removed: "TP: PV- / MID / PV+"
Changed lines of the file:
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@@
 		(uuid "cell-divider-v03")
 	)
-	(gr_text "ICARUS - 1U SOLAR PANEL PCB - 2S1P BASELINE"
+	(gr_text "ICARUS - 1U SOLAR PANEL PCB - 1S2P PARALLEL"
 		(at 105 107 0)
 		(layer "F.SilkS")
@@
 		(effects (font (size 0.8 0.8) (thickness 0.12)))
 	)
-	(gr_text "TP: PV- / MID / PV+"
+	(gr_text "TP: PV- / PV+"
 		(at 105 134.6 0)
 		(layer "F.Fab")
