File: hardware/ICARUS_1U_Solar_Panel_PCB_v0p7.kicad_sch (KiCad schematic)
At the start: 13 parts, among them J1 Molex_53398-0471

Commit message: Switch to parallel topology (1S2P) for v0.7
Lead-team-driven topology change. Both cells now share PANEL_POS and
PANEL_NEG nets (was 2S1P with intermediate SERIES_MID). J1 (Molex)
moved from F.Cu to B.Cu (bottom side, as instructed). Re-routed for
parallel: left B.Cu corridor (x=70) ties the two PANEL_NEG tab buses;
right B.Cu corridor (x=137) ties the two PANEL_POS centre buses; both
land on the bottom J1 pads. TP3/TP5 stay on F.Cu under SC2 (PANEL_POS
on PANEL_POS) to avoid crossing the B.Cu PANEL_NEG corridor.

Also removed: D1 (TVS DNP) and TP2 (SERIES_MID test pad), both obsolete
in 1S2P. SERIES_MID net dropped from the PCB net table.

Rename of v0p6.* -> v0p7.* across .kicad_sch / .kicad_pcb / .kicad_pro.

DRC parity clean: 0 errors / 0 unconnected / 0 parity / 0 shorts.
11 warnings = same library waivers as v0.6 (minus the D1/TP2 ones).

Co-Authored-By: Claude Opus 4.7 <noreply@anthropic.com>
Parts:
- removed D1: TVS_OPTIONAL_DNP, Diode_SMD:D_SOD-123, symbol ICARUS:TVS_DNP_2Pin
- removed TP2: SERIES_MID, TestPoint:TestPoint_Pad_D2.0mm, symbol ICARUS:TestPoint_1Pin
Connections:
- net PANEL_NEG: now also SC2.1 (NEG)
- net PANEL_POS: now also SC1.2 (POS)
- removed net SERIES_MID: SC1.2 (POS), SC2.1 (NEG)
Other:
- note added: "1S2P baseline (v0.7): SC1_NEG and SC2_NEG -> PANEL_NEG; SC1_POS and SC2_POS -> PANEL_POS. Cells in parallel; eliminates Voc OVP risk. Validate actual cell polarity before assembly."
- note added: "PCB v0.7 includes TP_NEG and TP_POS. J1 (Molex) is mounted on B.Cu (bottom). BENCH_ONLY_PANEL_NEG/BENCH_ONLY_PANEL_POS are fallback bench solder pads only; final interface is J1/harness."
- note removed: "2S1P baseline: SC1_NEG -> PANEL_NEG; SC1_POS -> SERIES_MID; SC2_NEG -> SERIES_MID; SC2_POS -> PANEL_POS. Validate actual cell polarity before assembly."
- note removed: "PCB v0.6 includes TP_NEG, TP_MID and TP_POS. BENCH_ONLY_PANEL_NEG/BENCH_ONLY_PANEL_POS are fallback bench solder pads only; final interface is J1/harness."
Changed lines of the file:
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@@
 	(wire (pts (xy 125.73 87.63) (xy 111.76 87.63)) (stroke (width 0) (type default)))
 	(wire (pts (xy 125.73 90.17) (xy 111.76 90.17)) (stroke (width 0) (type default)))
-	(wire (pts (xy 125.73 106.68) (xy 120.65 106.68)) (stroke (width 0) (type default)))
-	(wire (pts (xy 135.89 106.68) (xy 140.97 106.68)) (stroke (width 0) (type default)))
 	(global_label "PANEL_NEG" (shape input) (at 95.25 76.2 0) (fields_autoplaced) (effects (font (size 1.27 1.27)) (justify left)))
-	(global_label "SERIES_MID" (shape input) (at 95.25 78.74 0) (fields_autoplaced) (effects (font (size 1.27 1.27)) (justify left)))
-		(global_label "SERIES_MID" (shape input) (at 95.25 91.44 0) (fields_autoplaced) (effects (font (size 1.27 1.27)) (justify left)))
+	(global_label "PANEL_POS" (shape input) (at 95.25 78.74 0) (fields_autoplaced) (effects (font (size 1.27 1.27)) (justify left)))
+		(global_label "PANEL_NEG" (shape input) (at 95.25 91.44 0) (fields_autoplaced) (effects (font (size 1.27 1.27)) (justify left)))
 		(global_label "PANEL_POS" (shape input) (at 95.25 93.98 0) (fields_autoplaced) (effects (font (size 1.27 1.27)) (justify left)))
 	(global_label "PANEL_NEG" (shape input) (at 111.76 82.55 180) (fields_autoplaced) (effects (font (size 1.27 1.27)) (justify right)))
@@
 	(global_label "PANEL_POS" (shape input) (at 111.76 87.63 180) (fields_autoplaced) (effects (font (size 1.27 1.27)) (justify right)))
 	(global_label "PANEL_POS" (shape input) (at 111.76 90.17 180) (fields_autoplaced) (effects (font (size 1.27 1.27)) (justify right)))
-		(global_label "PANEL_NEG" (shape input) (at 120.65 106.68 180) (fields_autoplaced) (effects (font (size 1.27 1.27)) (justify right)))
-		(global_label "PANEL_POS" (shape input) (at 140.97 106.68 0) (fields_autoplaced) (effects (font (size 1.27 1.27)) (justify left)))
 		(global_label "PANEL_NEG" (shape input) (at 154.94 76.2 0) (fields_autoplaced) (effects (font (size 1.27 1.27)) (justify left)))
-			(global_label "SERIES_MID" (shape input) (at 154.94 83.82 0) (fields_autoplaced) (effects (font (size 1.27 1.27)) (justify left)))
 			(global_label "PANEL_POS" (shape input) (at 154.94 91.44 0) (fields_autoplaced) (effects (font (size 1.27 1.27)) (justify left)))
 			(global_label "PANEL_NEG" (shape input) (at 154.94 101.6 0) (fields_autoplaced) (effects (font (size 1.27 1.27)) (justify left)))
 			(global_label "PANEL_POS" (shape input) (at 154.94 109.22 0) (fields_autoplaced) (effects (font (size 1.27 1.27)) (justify left)))
-		(text "2S1P baseline: SC1_NEG -> PANEL_NEG; SC1_POS -> SERIES_MID; SC2_NEG -> SERIES_MID; SC2_POS -> PANEL_POS. Validate actual cell polarity before assembly." (at 67.31 57.15 0) (effects (font (size 1.27 1.27)) (justify left bottom)))
-	(text "PCB v0.6 includes TP_NEG, TP_MID and TP_POS. BENCH_ONLY_PANEL_NEG/BENCH_ONLY_PANEL_POS are fallback bench solder pads only; final interface is J1/harness." (at 67.31 61.0 0) (effects (font (size 1.27 1.27)) (justify left bottom)) (uuid "bench-note-v05"))
+		(text "1S2P baseline (v0.7): SC1_NEG and SC2_NEG -> PANEL_NEG; SC1_POS and SC2_POS -> PANEL_POS. Cells in parallel; eliminates Voc OVP risk. Validate actual cell polarity before assembly." (at 67.31 57.15 0) (effects (font (size 1.27 1.27)) (justify left bottom)))
+	(text "PCB v0.7 includes TP_NEG and TP_POS. J1 (Molex) is mounted on B.Cu (bottom). BENCH_ONLY_PANEL_NEG/BENCH_ONLY_PANEL_POS are fallback bench solder pads only; final interface is J1/harness." (at 67.31 61.0 0) (effects (font (size 1.27 1.27)) (justify left bottom)) (uuid "bench-note-v05"))
 	(symbol (lib_id "ICARUS:Solar_Cell_2Pin") (at 76.2 77.47 0) (unit 1) (exclude_from_sim no) (in_bom yes) (on_board yes) (dnp no)
 		(property "Reference" "SC1" (at 76.2 71.12 0) (effects (font (size 1.27 1.27))))
@@
 		(pin "4")
 	)
-		(symbol (lib_id "ICARUS:TVS_DNP_2Pin") (at 130.81 106.68 0) (unit 1) (exclude_from_sim no) (in_bom no) (on_board yes) (dnp yes)
-			(property "Reference" "D1" (at 130.81 101.0 0) (effects (font (size 1.27 1.27))))
-			(property "Value" "TVS_OPTIONAL_DNP" (at 130.81 112.0 0) (effects (font (size 1.27 1.27))))
-			(property "Footprint" "Diode_SMD:D_SOD-123" (at 130.81 115.0 0) (effects (font (size 1.27 1.27)) hide))
-			(pin "1")
-			(pin "2")
-		)
 		(symbol (lib_id "ICARUS:TestPoint_1Pin") (at 160.02 76.2 0) (unit 1) (exclude_from_sim no) (in_bom yes) (on_board yes) (dnp no)
 			(property "Reference" "TP1" (at 160.02 73.66 0) (effects (font (size 1.27 1.27))))
@@
 			(pin "1")
 		)
-			(symbol (lib_id "ICARUS:TestPoint_1Pin") (at 160.02 83.82 0) (unit 1) (exclude_from_sim no) (in_bom yes) (on_board yes) (dnp no)
-				(property "Reference" "TP2" (at 160.02 81.28 0) (effects (font (size 1.27 1.27))))
-				(property "Value" "SERIES_MID" (at 160.02 86.36 0) (effects (font (size 1.27 1.27))))
-				(property "Footprint" "TestPoint:TestPoint_Pad_D2.0mm" (at 160.02 88.9 0) (effects (font (size 1.27 1.27)) hide))
-			(pin "1")
-		)

Commit message: v0.7 cleanup: purge stale 2S1P / SERIES_MID / D1 / v0.6 references
The previous v0.7 merge left several stale strings hardcoded inside
files that the GUI still surfaced as if the board were still 2S1P.
This pass catches them all:

- PCB title block: v0.6 -> v0.7, "2S1P baseline" -> "1S2P parallel; J1 on B.Cu".
- Schematic title block: same v0.6 -> v0.7 / 2S1P -> 1S2P update.
- Schematic lib_symbols: drop the unused TVS_DNP_2Pin definition
  (D1 was removed in v0.7; the lib stub is now dead code).
- README.md: full rewrite for v0.7 — file paths v0p6 -> v0p7, the
  parameter tables now show Voc_panel = 2.70 V (1S2P, no overvoltage),
  the SC1_POS / SC2_NEG entries now point at PANEL_POS / PANEL_NEG
  (no SERIES_MID), the "Risco principal" Voc-OVP table is gone and
  replaced with a 1S2P-margins table, EPS limits row labels UVLO
  and OVP-trigger explicitly.
- Add SUPERSEDED banners to docs/CORRECAO_TOPOLOGIA_SERIE_v0p6.md,
  docs/REVIEW_ACTIONS_v0p6.md, docs/VALIDACAO_LOCAL_v0p6.md,
  docs/CELL_UNDER_COPPER_RISK_v0p6.md (partially) and a "still valid"
  note to docs/MECHANICAL_CELL_CLEARANCE_v0p6.md.
- Remove PR_BODY_v0p6.md (we merged v0.6 directly to main, no PR was
  opened, the file was a stranded artifact).
- Regenerate ERC/DRC reports and SVG plots — 0 errors / 0 parity
  preserved, only the title-block strings changed in the plot output.

Co-Authored-By: Claude Opus 4.7 <noreply@anthropic.com>
Other:
- title: ICARUS 1U Solar Panel Electrical Schematic v0.6 -> ICARUS 1U Solar Panel Electrical Schematic v0.7
Changed lines of the file:
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@@
 	(paper "A4")
 	(title_block
-		(title "ICARUS 1U Solar Panel Electrical Schematic v0.6")
-		(date "2026-05-24")
-		(rev "0.6-internal-review")
+		(title "ICARUS 1U Solar Panel Electrical Schematic v0.7")
+		(date "2026-05-28")
+		(rev "0.7")
 		(company "Porto Space Team - ICARUS")
-		(comment 1 "Baseline: 2S1P, TJ3xSCA-4080 Type 32")
+		(comment 1 "Baseline: 1S2P (parallel), TJ3xSCA-4080 Type 32")
 		(comment 2 "EPS I solar connector: pins 1/2 PV-, pins 3/4 PV+")
 	)
