File: hardware/ICARUS_1U_Solar_Panel_PCB_v0p7.kicad_sch (KiCad schematic)
At the start: 11 parts, among them J1 Molex_53398-0471

Commit message: Sync TP and MountingHole footprints with KiCad 10 stdlib (zeros 10 warnings)
Manually rewrote the 8 embedded footprints (TP1, TP3, TP4, TP5 +
H1-H4) to match the structure of the standard KiCad 10.0 library
versions in
  C:\Program Files\KiCad\10.0\share\kicad\footprints\TestPoint.pretty
  C:\Program Files\KiCad\10.0\share\kicad\footprints\MountingHole.pretty
preserving the instance-specific bits (uuid, position, reference,
pad net assignments).

Schematic: set TP1 and TP3 to in_bom=no to match the stdlib
TestPoint_Pad_D2.0mm attr exclude_from_bom (test pads are not
purchasable components — they are built into the PCB).

DRC result:
- v0.6: 13 warnings (3 lib + 10 lib_mismatch)
- v0.7 before this commit: 11 warnings (D1 + TP2 already removed)
- v0.7 now: 3 warnings (only lib_footprint_issues from CLI not
  resolving ICARUS_Solar / ICARUS_Connector local libs).

All 10 lib_footprint_mismatch warnings cleared.

Co-Authored-By: Claude Opus 4.7 <noreply@anthropic.com>
Parts:
- TP1, TP3: now left out of the parts list
Changed lines of the file:
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@@
 		(pin "4")
 	)
-		(symbol (lib_id "ICARUS:TestPoint_1Pin") (at 160.02 76.2 0) (unit 1) (exclude_from_sim no) (in_bom yes) (on_board yes) (dnp no)
+		(symbol (lib_id "ICARUS:TestPoint_1Pin") (at 160.02 76.2 0) (unit 1) (exclude_from_sim no) (in_bom no) (on_board yes) (dnp no)
 			(property "Reference" "TP1" (at 160.02 73.66 0) (effects (font (size 1.27 1.27))))
 			(property "Value" "PANEL_NEG" (at 160.02 78.74 0) (effects (font (size 1.27 1.27)) (hide yes)))
@@
 			(pin "1")
 		)
-			(symbol (lib_id "ICARUS:TestPoint_1Pin") (at 160.02 91.44 0) (unit 1) (exclude_from_sim no) (in_bom yes) (on_board yes) (dnp no)
+			(symbol (lib_id "ICARUS:TestPoint_1Pin") (at 160.02 91.44 0) (unit 1) (exclude_from_sim no) (in_bom no) (on_board yes) (dnp no)
 				(property "Reference" "TP3" (at 160.02 88.9 0) (effects (font (size 1.27 1.27))))
 				(property "Value" "PANEL_POS" (at 160.02 93.98 0) (effects (font (size 1.27 1.27)) (hide yes)))
